File: esp32.sch (KiCad schematic (older format))
At the start: 34 parts

Commit message: finished schematic, first placement started
Parts:
- C1: renamed from C?; value 100n -> 100n/25V; footprint (none) -> bytewerk_capacitors:C_0603_1608Metric
- C2, C4, C6, C7: renamed from C?; footprint (none) -> bytewerk_capacitors:C_0603_1608Metric
- C3, C5: renamed from C?; footprint (none) -> bytewerk_capacitors:C_0805_2012Metric
- D1, D2: renamed from D?; footprint (none) -> LED_SMD:LED_0805_2012Metric
- J1: renamed from J?; footprint (none) -> Connector_PinHeader_2.54mm:PinHeader_1x02_P2.54mm_Horizontal
- J2: renamed from J?; value Micro_SD_Card_Det -> DM3AT-SF-PEJM5(40); footprint (none) -> Connector_Card:microSD_HC_Hirose_DM3AT-SF-PEJM5
- L1, L2: renamed from L?; footprint (none) -> Inductor_SMD:L_0603_1608Metric
- R1, R10, R11, R12, R13, R14, R15, R16, R17, R2, R3, R4, R5, R6, R7, R8, R9: renamed from R?; footprint (none) -> bytewerk_resistors:R_0603_1608Metric
- Y1: renamed from Y?; value Crystal -> LFXTAL009709Bulk; footprint (none) -> Crystal:Crystal_SMD_3215-2Pin_3.2x1.5mm
- gave numbers to parts that had none: 3
Connections:
- wire segments 132 -> 133
