File: esp32_can_donlge.kicad_pcb (KiCad board)
At the start: 2 copper layers, 0 parts

Commit message: finished schematic, first placement started
Parts:
- added C1: 100n/25V, bytewerk_capacitors:C_0603_1608Metric, F.Cu at (164.4, 103.8)
- added C10: 10u/25V, bytewerk_capacitors:C_0805_2012Metric, F.Cu at (197.6, 85.9)
- added C11: 1u/25V, bytewerk_capacitors:C_0603_1608Metric, F.Cu at (186.2, 85.1)
- added C12: 10n/25V, bytewerk_capacitors:C_0603_1608Metric, F.Cu at (195.5, 86.1)
- added C13: 100n/25V, bytewerk_capacitors:C_0603_1608Metric, F.Cu at (186.9, 82.7)
- added C14: 10p/50V, bytewerk_capacitors:C_0603_1608Metric, F.Cu at (191.0, 89.3)
- added C15: 10u/25V, bytewerk_capacitors:C_0805_2012Metric, F.Cu at (181.9, 79.9)
- added C16: 10u/25V, bytewerk_capacitors:C_0805_2012Metric, F.Cu at (179.7, 79.9)
- added C17: 100n/10V, bytewerk_capacitors:C_0603_1608Metric, F.Cu at (167.0, 64.7)
- added C18: 4u7/10V, bytewerk_capacitors:C_0805_2012Metric, F.Cu at (170.5, 64.4)
- added C19: 100n/25V, bytewerk_capacitors:C_0603_1608Metric, F.Cu at (170.9, 72.4)
- added C2: 100n/25V, bytewerk_capacitors:C_0603_1608Metric, B.Cu at (188.9, 102.6)
- added C20: 4u7/10V, bytewerk_capacitors:C_0805_2012Metric, F.Cu at (170.7, 74.3)
- added C3: 10u/25V, bytewerk_capacitors:C_0805_2012Metric, B.Cu at (190.8, 102.6)
- added C4: 100n/25V, bytewerk_capacitors:C_0603_1608Metric, F.Cu at (160.9, 103.8)
- added C5: 10u/25V, bytewerk_capacitors:C_0805_2012Metric, F.Cu at (161.0, 105.8)
- added C6: C, bytewerk_capacitors:C_0603_1608Metric, F.Cu at (167.7, 106.5)
- added C7: C, bytewerk_capacitors:C_0603_1608Metric, F.Cu at (173.7, 106.5)
- added C8: 100n/25V, bytewerk_capacitors:C_0603_1608Metric, F.Cu at (188.5, 96.6)
- added C9: 10u/25V, bytewerk_capacitors:C_0805_2012Metric, F.Cu at (186.2, 96.6)
- added D1: LED, LED_SMD:LED_0805_2012Metric, F.Cu at (188.6, 73.7)
- added D2: LED, LED_SMD:LED_0805_2012Metric, F.Cu at (192.2, 73.7)
- added D3: BAT54C, Package_TO_SOT_SMD:SOT-23, B.Cu at (189.1, 68.0)
- added D4: NUP2105L, Package_TO_SOT_SMD:SOT-23, B.Cu at (200.5, 99.7)
- added D5: B130-E3, Diode_SMD:D_SMA, B.Cu at (203.8, 89.7)
- added D6: LED, LED_SMD:LED_0805_2012Metric, F.Cu at (182.0, 73.7)
- added D7: LED, LED_SMD:LED_0805_2012Metric, F.Cu at (184.9, 73.7)
- added J1: Conn_01x02_Male, Connector_PinHeader_2.54mm:PinHeader_1x02_P2.54mm_Horizontal, B.Cu at (183.9, 64.3)
- added J2: DM3AT-SF-PEJM5(40), Connector_Card:microSD_HC_Hirose_DM3AT-SF-PEJM5, B.Cu at (173.6, 92.3)
- added J3: DB9_Male, Connector_Dsub:DSUB-9_Male_EdgeMount_P2.77mm, F.Cu at (206.4, 99.3)
- added J4: USB_B_Micro, Connector_USB:USB_Micro-B_Wuerth_629105150521_CircularHoles, F.Cu at (161.4, 69.1)
- added L1: L, Inductor_SMD:L_0603_1608Metric, B.Cu at (192.9, 102.6)
- added L2: L, Inductor_SMD:L_0603_1608Metric, B.Cu at (181.0, 83.5)
- added L3: XFL3012-222ME, bytewerk-inductors:L_Coilcraft_XLF3012, F.Cu at (185.3, 79.9)
- added L4: L, Inductor_SMD:L_0603_1608Metric, F.Cu at (166.6, 73.7)
- added L5: L, Inductor_SMD:L_0805_2012Metric, F.Cu at (166.9, 66.9)
- added Q1: DMG2305UX-7, Package_TO_SOT_SMD:SOT-23, B.Cu at (195.6, 102.7)
- added Q2: BC817, Package_TO_SOT_SMD:SOT-23, B.Cu at (185.4, 71.7)
- added Q3: BC817, Package_TO_SOT_SMD:SOT-23, B.Cu at (185.4, 68.0)
- added R1: 1k, bytewerk_resistors:R_0603_1608Metric, F.Cu at (188.6, 70.1)
- added R10: 10R, bytewerk_resistors:R_0603_1608Metric, B.Cu at (184.8, 94.2)
- added R11: 33R, bytewerk_resistors:R_0603_1608Metric, B.Cu at (184.8, 97.6)
- added R12: 33R, bytewerk_resistors:R_0603_1608Metric, B.Cu at (184.8, 89.1)
- added R13: 33R, bytewerk_resistors:R_0603_1608Metric, B.Cu at (184.8, 92.5)
- added R14: 200R, bytewerk_resistors:R_0603_1608Metric, B.Cu at (184.8, 95.9)
- added R15: 10k, bytewerk_resistors:R_0603_1608Metric, B.Cu at (184.8, 99.3)
- added R16: 220R, bytewerk_resistors:R_0603_1608Metric, F.Cu at (166.6, 79.7)
- added R17: 220R, bytewerk_resistors:R_0603_1608Metric, F.Cu at (162.8, 79.7)
- added R18: 0R, bytewerk_resistors:R_0603_1608Metric, F.Cu at (195.9, 92.9)
- added R19: 10k, bytewerk_resistors:R_0603_1608Metric, F.Cu at (191.3, 100.4)
- added R2: 1k, bytewerk_resistors:R_0603_1608Metric, F.Cu at (192.2, 70.1)
- added R20: 10k, bytewerk_resistors:R_0603_1608Metric, F.Cu at (194.5, 100.4)
- added R21: 1k, bytewerk_resistors:R_0603_1608Metric, F.Cu at (199.3, 94.4)
- added R22: 470R, bytewerk_resistors:R_0603_1608Metric, F.Cu at (194.5, 102.2)
- added R23: 100R, bytewerk_resistors:R_0603_1608Metric, F.Cu at (200.1, 98.5)
- added R24: 1M, bytewerk_resistors:R_0603_1608Metric, F.Cu at (197.4, 82.4)
- added R25: 120k, bytewerk_resistors:R_0603_1608Metric, F.Cu at (195.6, 82.4)
- added R26: 82k, bytewerk_resistors:R_0603_1608Metric, B.Cu at (205.0, 86.6)
- added R27: 33k, bytewerk_resistors:R_0603_1608Metric, B.Cu at (201.7, 86.6)
- added R28: n.b., bytewerk_resistors:R_0603_1608Metric, F.Cu at (199.2, 82.4)
- added R29: 18k, bytewerk_resistors:R_0603_1608Metric, F.Cu at (186.2, 86.8)
- added R3: 10k, bytewerk_resistors:R_0603_1608Metric, F.Cu at (164.4, 105.8)
- added R30: 200R, bytewerk_resistors:R_0603_1608Metric, F.Cu at (186.2, 88.5)
- added R31: 82k, bytewerk_resistors:R_0603_1608Metric, B.Cu at (195.5, 86.1)
- added R32: 1M, bytewerk_resistors:R_0603_1608Metric, F.Cu at (192.8, 89.3)
- added R33: 309k, bytewerk_resistors:R_0603_1608Metric, F.Cu at (194.5, 89.3)
- added R34: 22k, bytewerk_resistors:R_0603_1608Metric, F.Cu at (174.2, 73.6)
- added R35: 47k, bytewerk_resistors:R_0603_1608Metric, F.Cu at (177.8, 73.6)
- added R36: 1k, bytewerk_resistors:R_0603_1608Metric, F.Cu at (174.2, 71.7)
- added R37: 1k, bytewerk_resistors:R_0603_1608Metric, F.Cu at (182.0, 70.1)
- added R38: 1k, bytewerk_resistors:R_0603_1608Metric, F.Cu at (184.9, 70.1)
- added R39: 1k, bytewerk_resistors:R_0603_1608Metric, B.Cu at (181.6, 70.6)
- added R4: 10k, bytewerk_resistors:R_0603_1608Metric, B.Cu at (198.5, 102.7)
- added R40: 1k, bytewerk_resistors:R_0603_1608Metric, B.Cu at (181.6, 68.7)
- added R5: 10k, bytewerk_resistors:R_0603_1608Metric, B.Cu at (190.1, 90.8)
- added R6: 10k, bytewerk_resistors:R_0603_1608Metric, B.Cu at (190.1, 92.5)
- added R7: 10k, bytewerk_resistors:R_0603_1608Metric, B.Cu at (190.1, 95.9)
- added R8: 10k, bytewerk_resistors:R_0603_1608Metric, B.Cu at (190.1, 97.6)
- added R9: 33R, bytewerk_resistors:R_0603_1608Metric, B.Cu at (184.8, 90.8)
- added U1: ESP32-WROOM-32, bytewerk-esp32:ESP32-WROOM-32, F.Cu at (165.4, 92.3)
- added U2: SN65HVD230DR, Package_SO:SOIC-8_3.9x4.9mm_P1.27mm, F.Cu at (193.6, 96.6)
- added U3: TLP175A, Package_SO:MFSOP6-4_4.4x3.6mm_P1.27mm, F.Cu at (200.6, 101.7)
- added U4: LT8607, Package_SO:MSOP-10-1EP_3x3mm_P0.5mm_EP1.68x1.88mm, F.Cu at (191.4, 84.6)
- added U5: USBLC6-2SC6, Package_TO_SOT_SMD:SOT-23-6, F.Cu at (167.1, 69.8)
- added U6: CP2102N-A01-GQFN24, Package_DFN_QFN:QFN-24-1EP_4x4mm_P0.5mm_EP2.6x2.6mm, F.Cu at (175.3, 67.3)
- added Y1: LFXTAL009709Bulk, Crystal:Crystal_SMD_3215-2Pin_3.2x1.5mm, F.Cu at (170.7, 105.4)
Other:
- copper layers 2 -> 4
