File: esp32_can_donlge.sch (KiCad schematic (older format))
At the start: 0 parts

Commit message: finished schematic, first placement started
Connections:
- wire segments 14 -> 17
Changed lines of the file:
@@
 F2 "CAN_P" B R 6450 1750 50
 F3 "CAN_N" B R 6450 1850 50
+F4 "Power_Good" O R 6450 1950 50
 $EndSheet
 $Sheet
@@
 Wire Wire Line
 	3750 3800 4800 3800
+Wire Wire Line
+	6450 1950 6800 1950
+Wire Wire Line
+	6800 1950 6800 3300
+Wire Wire Line
+	6800 3300 6450 3300
 $EndSCHEMATC
