File: power_supply.sch (KiCad schematic (older format))
At the start: 9 parts

Commit message: finished schematic, first placement started
Parts:
- removed D?: 1N5822, Diode_THT:D_DO-201AD_P15.24mm_Horizontal, symbol Diode:1N5822
- removed U?: NCP718BSN330T1G, Package_TO_SOT_SMD:TSOT-23-5, symbol bytewerk-vreg:NCP718BSN330T1G
- added C11: 1u/25V, bytewerk_capacitors:C_0603_1608Metric, symbol bytewerk-discrete:C
- added C12: 10n/25V, bytewerk_capacitors:C_0603_1608Metric, symbol bytewerk-discrete:C
- added C14: 10p/50V, bytewerk_capacitors:C_0603_1608Metric, symbol bytewerk-discrete:C
- added C16: 10u/25V, bytewerk_capacitors:C_0805_2012Metric, symbol bytewerk-discrete:C
- added D5: B130-E3, Diode_SMD:D_SMA, symbol Diode:B130-E3
- added L3: XFL3012-222ME, bytewerk-inductors:L_Coilcraft_XLF3012, symbol Device:L
- added R24, R32: 1M, bytewerk_resistors:R_0603_1608Metric, symbol bytewerk-discrete:R
- added R25: 120k, bytewerk_resistors:R_0603_1608Metric, symbol bytewerk-discrete:R
- added R28: n.b., bytewerk_resistors:R_0603_1608Metric, symbol bytewerk-discrete:R
- added R29: 18k, bytewerk_resistors:R_0603_1608Metric, symbol bytewerk-discrete:R
- added R30: 200R, bytewerk_resistors:R_0603_1608Metric, symbol bytewerk-discrete:R
- added R31: 82k, bytewerk_resistors:R_0603_1608Metric, symbol bytewerk-discrete:R
- added R33: 309k, bytewerk_resistors:R_0603_1608Metric, symbol bytewerk-discrete:R
- added U4: LT8607, Package_SO:MSOP-10-1EP_3x3mm_P0.5mm_EP1.68x1.88mm, symbol bytewerk-vreg:LT8607
- C10, C15: renamed from C?; footprint (none) -> bytewerk_capacitors:C_0805_2012Metric
- C13: renamed from C?; footprint (none) -> bytewerk_capacitors:C_0603_1608Metric
- J3: renamed from J?; footprint (none) -> Connector_Dsub:DSUB-9_Male_EdgeMount_P2.77mm
- R26, R27: renamed from R?; footprint (none) -> bytewerk_resistors:R_0603_1608Metric
- gave numbers to parts that had none: 1
Connections:
- net labels added: Power_Good, V_BAT
- wire segments 33 -> 80
Other:
- note added: "Voltage regulator will be \nshut down below 9V of V_BAT\nVin(en) around 9,33V"
